File: Hardware/Schematic.sch (EAGLE design)
At the start: 105 parts, among them IC1 BQ25180YBGR, IC2 DRV2605YZFR, IC3 BMA421, IC9 RT6160AWSC, J1 503480-2400, J2 TC2030-IDC, J4 KH-TYPE-C-16P, Q1 20V/4.2A/52mΩ/1.4W, Q3 SI1308EDL-T1-GE3, U1 NRF52840 _QF, U3 MAX17048G+T10, X1 32MHz, X2 32.768KHz

Commit message: solve sugestion from issue #3
Parts:
- C42: device InkTime_v5:GRM011R60J152KE01L_2_GRM011R60J152KE01L -> Libraria_DANI:GRM011R60J152KE01L_2_GRM011R60J152KE01L
- C43, EPD_C1, EPD_C10, EPD_C11, EPD_C12, EPD_C2, EPD_C6, EPD_C7, EPD_C8, EPD_C9: device InkTime_v5:NORDIC_NRF_3_CAPACITOR_0402_L -> Libraria_DANI:NORDIC_NRF_3_CAPACITOR_0402_L
- EPD_C5: device InkTime_v5:NORDIC_NRF_3_CAPACITOR_0201_L -> Libraria_DANI:NORDIC_NRF_3_CAPACITOR_0201_L
- R1_USB, R2_USB: device InkTime_v5:CPF0201D7K68C1_CPF0201D7K68C1 -> Libraria_DANI:CPF0201D7K68C1_CPF0201D7K68C1
